File: 16x2/TB EAGLE/PB/SerLCD_16x4_pb-v01.brd (EAGLE design)
At the start: 87.7 x 133.3 mm, 22 parts

Commit message: Some library work, and the 16x4 is almost done
Parts:
- removed J4, J5, J6: (no value), SparkFun-Connectors:1X01_OFFSET
- removed U$1: 3.3V Flying Jalapeno, Testing-8-24-15:FLYING_JALAPENO_V2_M
- removed U$10: 74LVC4066_MUX_1:1_X4, Testing:SO14
- added JP1: MISO, SparkFun-Jumpers:SMT-JUMPER_2_NC_PASTE_NO-SILK
- added JP2: SCK, SparkFun-Jumpers:SMT-JUMPER_2_NC_PASTE_NO-SILK
- added JP3: RST, SparkFun-Jumpers:SMT-JUMPER_2_NC_PASTE_NO-SILK
- added JP4: MOSI, SparkFun-Jumpers:SMT-JUMPER_2_NC_PASTE_NO-SILK
- added R1, R2: 10k, SparkFun-Resistors:0603
- added U1: 5V Flying Jalapeno, Testing:FLYING_JALAPENO_V2_M
- added U2: 74LVC4066_MUX_1:1_X4, Testing:SO14
- J1: value (none) -> AVR_PROG; device SparkFun-Connectors:1X01_OFFSET -> SparkFun-Connectors:2X3_LOCK
- J2: device SparkFun-Connectors:1X01_OFFSET -> SparkFun-Connectors:1X06_LOCK
- J3: value (none) -> SER_LCD16X2; device SparkFun-Connectors:1X01_OFFSET -> SerLCD_dimensions:SER_LCD_16X2
- moved J3 92.3 mm to (63.5, 29.2), turned to 90 degrees
- moved J1 66.5 mm to (6.35, 124.5), turned to 90 degrees
- moved J2 34.7 mm to (10.2, 74.9), turned to 270 degrees
- moved U$2 11.4 mm to (83.8, 141.0)
- moved U$6 11.4 mm to (0.00, 99.1)
- moved U$9 11.4 mm to (3.81, 141.0)
- moved U$3 11.4 mm to (83.8, 114.3)
Connections:
- removed net BATT3V_TP: U$1.3, U$1.33
- removed net BRD_RST: J3.1
- removed net BRD_VCC: J2.1, U$1.38
- removed net PGM_SWTICH_EN: U$1.60, U$10.12, U$10.13, U$10.5, U$10.6
- new net 3.3_VCC: J1.2, J3.P$3, R1.2
- new net CS: J3.P$10, U1.60
- new net DTR_FJ: J2.1, J3.P$6, U1.14
- new net MISO: J3.P$8, JP1.2, U1.29, U2.2
- new net MISO_P: J1.1, JP1.1, U2.1
- new net MOSI: J3.P$9, JP4.2, U1.59, U2.10
- new net MOSI_P: J1.4, JP4.1, U2.11
- new net N$7: R1.1, R2.2, U1.38
- new net PGM_SWITCH_EN: U1.28, U2.12, U2.13, U2.5, U2.6
- new net RAW_VIA_V2: J3.P$15, J3.P$17, U1.3, U1.33
- new net RST: J3.P$20, JP3.2, U2.9
- new net RST_P: J1.5, JP3.1, U2.8
- new net RX1_FJ: J2.2, J3.P$12, J3.P$5, U1.52
- new net SCK: J3.P$7, JP2.2, U1.30, U2.3
- new net SCK_P: J1.3, JP2.1, U2.4
- new net SCL: J3.P$13, U1.53
- new net SDA: J3.P$14, U1.23
- new net TX1_FJ: J2.3, J3.P$11, J3.P$19, J3.P$4, U1.22
- net 5V_VIN: now also U1.2, U1.32, U2.14; no longer U$1.2, U$1.32, U$10.14
- net GND: now also J1.6, J2.5, J2.6, J3.P$1, J3.P$16, J3.P$18, J3.P$2, R2.1, U1.1, U1.31, U2.7; no longer J1.1, U$1.1, U$1.31, U$10.7
- net N$1: now also U1.5; no longer U$1.5
- net N$2: now also U1.58; no longer U$1.58
- net N$3: now also U1.7; no longer U$1.7
- net N$4: now also U1.36; no longer U$1.36
- net N$5: now also U1.35; no longer U$1.35
- net N$6: now also U1.6; no longer U$1.6
Other:
- board size 87.7 x 133.3 mm -> 87.7 x 144.8 mm
- board text added: "10K"
