File: 16x2/TB EAGLE/PB/SerLCD_16x4_pb-v01.sch (EAGLE design)
At the start: 16 parts

Commit message: Some library work, and the 16x4 is almost done
Parts:
- removed J4, J5, J6: (no value), SparkFun-Connectors:CONN_01OFFSET
- removed U$1: 3.3V Flying Jalapeno, Testing-8-24-15:FLYING_JALAPENO_V2MALE
- removed U$10: 74LVC4066_MUX_1:1_X4, Testing:74LVC4066_MUX_1:1_X4
- added JP1: MISO, SparkFun-Jumpers:JUMPER-SMT_2_NC_PASTE_NO-SILK
- added JP2: SCK, SparkFun-Jumpers:JUMPER-SMT_2_NC_PASTE_NO-SILK
- added JP3: RST, SparkFun-Jumpers:JUMPER-SMT_2_NC_PASTE_NO-SILK
- added JP4: MOSI, SparkFun-Jumpers:JUMPER-SMT_2_NC_PASTE_NO-SILK
- added R1, R2: 10k, SparkFun-Resistors:10KOHM-0603-1/10W-1%
- added U1: 5V Flying Jalapeno, Testing:FLYING_JALAPENO_V2MALE
- added U2: 74LVC4066_MUX_1:1_X4, Testing:74LVC4066_MUX_1:1_X4
- J1: value (none) -> AVR_PROG; device SparkFun-Connectors:CONN_01OFFSET -> SparkFun-Connectors:AVR_SPI_PROG_3X22X3_LOCK
- J2: device SparkFun-Connectors:CONN_01OFFSET -> SparkFun-Connectors:6_PIN_SERIAL_TARGETLOCK
- J3: value (none) -> SER_LCD16X2; device SparkFun-Connectors:CONN_01OFFSET -> SerLCD_dimensions:SER_LCD16X2
Connections:
- removed net BATT3V_TP: U$1.V2
- removed net BRD_RST: J3.1
- removed net BRD_VCC: J2.1, U$1.A2
- removed net PGM_SWTICH_EN: U$1.53, U$10.1E, U$10.2E, U$10.3E, U$10.4E
- new net 3.3_VCC: J1.2, J3.+, R1.2
- new net CS: J3./CS, U1.53(SS)
- new net DTR_FJ: J2.DTR, J3.R(DTR), U1.2(INT0)
- new net MISO: J3.SDO, JP1.2, U1.50(MISO), U2.1Z
- new net MISO_P: J1.1, JP1.1, U2.1Y
- new net MOSI: J3.SDI, JP4.2, U1.51(MOSI), U2.4Z
- new net MOSI_P: J1.4, JP4.1, U2.4Y
- new net N$7: R1.1, R2.2, U1.A2
- new net PGM_SWITCH_EN: U1.30, U2.1E, U2.2E, U2.3E, U2.4E
- new net RAW_VIA_V2: J3.5-12V, J3.RAW, U1.V2
- new net RST: J3.RST, JP3.2, U2.3Z
- new net RST_P: J1.5, JP3.1, U2.3Y
- new net RX1_FJ: J2.RXI, J3.TX, J3.TXO, U1.19(RX1/INT4)
- new net SCK: J3.SCK, JP2.2, U1.52(SCK), U2.2Z
- new net SCK_P: J1.3, JP2.1, U2.2Y
- new net SCL: J3.CL, U1.21(SCL/INT2)
- new net SDA: J3.DA, U1.20(SDA/INT3)
- new net TX1_FJ: J2.TXO, J3.RX, J3.RX@19, J3.RXI, U1.18(TX1/INT5)
- net 5V_VIN: now also U1.V1, U2.VCC; no longer U$1.V1, U$10.VCC
- net GND: now also J1.6, J2.CTS, J2.GND, J3.GND@1, J3.GND@16, J3.GND@18, J3.GND@2, R2.1, U1.GND, U2.GND; no longer J1.1, U$1.GND, U$10.GND
- net N$1: now also U1.CAP_PAD1; no longer U$1.CAP_PAD1
- net N$2: now also U1.CAP_PAD2; no longer U$1.CAP_PAD2
- net N$3: now also U1.43/PT_PASS; no longer U$1.43/PT_PASS
- net N$4: now also U1.42/PT_FAIL; no longer U$1.42/PT_FAIL
- net N$5: now also U1.40/FAIL; no longer U$1.40/FAIL
- net N$6: now also U1.41/PASS; no longer U$1.41/PASS
Other:
- note added: "Bypass switch jumpers"
- note added: "Flying Jalapeno (Testing Dev Board)"
- note added: "JUMPER to RAW"
- note added: "LCD connections (pogopins)"
- note added: "PROGRAMMING LINES"
- note added: "RAW INPUT 7V, 500mA"
- note added: "SERIAL UPLOAD"
- moved on the sheet: 1, 2, LED1, LED2, LED3, LED4
