File: 16x2/TB EAGLE/PB/SerLCD_16x2_pb-v01.brd (EAGLE design)
At the start: 73.7 x 139.7 mm, 21 parts, among them J1 AVR_PROG, J3 SER_LCD16X2, U1 5V Flying Jalapeno, U2 74LVC4066_MUX_1:1_X4

Commit message: added preTest to 3.3V on 16x2
This will also be used to verify that the vreg is outputing proper
voltage later in the test.

NOTE: I still need to add this to 20x4 version
Parts:
- removed R1, R2: 10k, SparkFun-Resistors:0603
- added R5, R6: 10K, SparkFun-Resistors:0603-RES
- added R7: 100k, SparkFun-Resistors:0603-RES
Connections:
- removed net N$7: R1.1, R2.2, U1.38
- new net PT_CTRL: R5.1, U1.44
- new net PT_READ_3.3V: R5.2, R6.1, R7.2, U1.40
- net 3.3_VCC: now also R6.2; no longer R1.2
- net GND: now also R7.1; no longer R2.1
Routing:
- net PT_READ_3.3V: track 0.00 -> 115.1 mm, vias 0 -> 2
- net N$7: track 105.7 -> 0.00 mm
- net PT_CTRL: track 0.00 -> 96.6 mm, vias 0 -> 4
- net N$3: track 131.9 -> 127.4 mm
Other:
- board text added: "100K"
Changed lines of the file:
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@@
 <layer number="26" name="bNames" color="7" fill="1" visible="no" active="yes"/>
 <layer number="27" name="tValues" color="7" fill="1" visible="no" active="yes"/>
-<layer number="28" name="bValues" color="7" fill="1" visible="no" active="yes"/>
+<layer number="28" name="bValues" color="7" fill="1" visible="yes" active="yes"/>
 <layer number="29" name="tStop" color="7" fill="3" visible="no" active="yes"/>
 <layer number="30" name="bStop" color="7" fill="6" visible="no" active="yes"/>
@@
 <text x="66.294" y="12.954" size="1.27" layer="21" font="vector" ratio="15">PASS</text>
 <text x="66.294" y="6.604" size="1.27" layer="21" font="vector" ratio="15">FAIL</text>
-<text x="37.719" y="44.45" size="0.8128" layer="22" font="vector" ratio="15" rot="MR0">10K</text>
-<text x="32.766" y="44.45" size="0.8128" layer="22" font="vector" ratio="15" rot="MR0">10K</text>
+<text x="37.846" y="44.196" size="0.8128" layer="22" font="vector" ratio="15" rot="MR0">10K</text>
+<text x="32.766" y="44.196" size="0.8128" layer="22" font="vector" ratio="15" rot="MR0">10K</text>
 <text x="1.524" y="130.175" size="0.8128" layer="21" font="vector" ratio="15">AVR ISP</text>
 <text x="15.24" y="64.77" size="0.8128" layer="21" font="vector" ratio="15" rot="R90">Serial upload</text>
 <text x="11.684" y="74.549" size="0.8128" layer="21" font="vector" ratio="15">DTR</text>
+<text x="33.274" y="37.592" size="0.8128" layer="22" font="vector" ratio="15" rot="MR0">100K</text>
 </plain>
 <attributes>
@@
 <attribute name="NAME" x="19.431" y="117.602" size="1.016" layer="26" font="vector" ratio="10" rot="MR90"/>
 </element>
-<element name="R1" library="SparkFun-Resistors" package="0603" value="10k" x="31.75" y="43.18" rot="MR0">
-<attribute name="PROD_ID" value="RES-00824" x="31.75" y="43.18" size="1.778" layer="28" font="vector" ratio="15" rot="MR0" display="off"/>
-</element>
-<element name="R2" library="SparkFun-Resistors" package="0603" value="10k" x="36.83" y="43.18" rot="MR0">
-<attribute name="PROD_ID" value="RES-00824" x="36.83" y="43.18" size="1.778" layer="28" font="vector" ratio="15" rot="MR0" display="off"/>
-</element>
 <element name="J3" library="SerLCD_dimensions" package="SER_LCD_16X2" value="SER_LCD16X2" x="57.15" y="29.21" rot="R90"/>
 <element name="J1" library="SparkFun-Connectors" package="2X3_LOCK" value="AVR_PROG" x="5.08" y="123.19" rot="R90"/>
@@
 <element name="JP4" library="SparkFun-Jumpers" package="SMT-JUMPER_2_NC_PASTE_NO-SILK" value="MOSI" x="20.32" y="121.92" rot="MR90"/>
 <element name="J2" library="SparkFun-Connectors" package="1X06_LOCK" value="" x="10.16" y="74.93" rot="R270"/>
+<element name="R5" library="SparkFun-Resistors" package="0603-RES" value="10K" x="36.83" y="43.18" rot="MR0">
+<attribute name="PROD_ID" value="RES-00824" x="36.83" y="43.18" size="1.778" layer="28" font="vector" ratio="15" rot="MR0" display="off"/>
+</element>
+<element name="R6" library="SparkFun-Resistors" package="0603-RES" value="10K" x="31.75" y="43.18" rot="MR0">
+<attribute name="PROD_ID" value="RES-00824" x="31.75" y="43.18" size="1.778" layer="28" font="vector" ratio="15" rot="MR0" display="off"/>
+</element>
+<element name="R7" library="SparkFun-Resistors" package="0603-RES" value="100k" x="31.75" y="39.37" rot="MR180">
+<attribute name="PROD_ID" value="RES-07828" x="31.75" y="39.37" size="1.778" layer="28" font="vector" ratio="15" rot="MR180" display="off"/>
+</element>
 </elements>
 <signals>
@@
 <contactref element="LED3" pad="C"/>
 <contactref element="U2" pad="7"/>
-<contactref element="R2" pad="1"/>
 <contactref element="J3" pad="P$16"/>
 <contactref element="J3" pad="P$1"/>
@@
 <via x="1.905" y="42.926" extent="1-16" drill="0.508"/>
 <via x="1.905" y="40.894" extent="1-16" drill="0.508"/>
+<contactref element="R7" pad="1"/>
 </signal>
 <signal name="5V_VIN" class="10">
@@
 <contactref element="LED1" pad="A"/>
 <wire x1="29.21" y1="53.975" x2="29.21" y2="11.43" width="0.254" layer="1"/>
-<wire x1="29.21" y1="133.0325" x2="29.21" y2="53.975" width="0.254" layer="16"/>
-<wire x1="21.59" y1="133.0325" x2="29.21" y2="133.0325" width="0.254" layer="16"/>
-<wire x1="20.0025" y1="134.62" x2="21.59" y2="133.0325" width="0.254" layer="16"/>
+<wire x1="29.21" y1="125.4125" x2="29.21" y2="53.975" width="0.254" layer="16"/>
+<wire x1="20.0025" y1="134.62" x2="29.21" y2="125.4125" width="0.254" layer="16"/>
 <wire x1="29.21" y1="11.43" x2="28.98" y2="11.43" width="0.254" layer="1"/>
 <wire x1="20.0025" y1="134.62" x2="19.83" y2="134.7" width="0.254" layer="16"/>
@@
 <wire x1="17.78" y1="134.9375" x2="17.83" y2="134.7" width="0.254" layer="16"/>
 <via x="66.9925" y="10.16" extent="1-16" drill="0.381"/>
-</signal>
-<signal name="N$7">
-<contactref element="U1" pad="38"/>
-<contactref element="R2" pad="2"/>
-<contactref element="R1" pad="1"/>
-<wire x1="35.98" y1="43.18" x2="32.6" y2="43.18" width="0.254" layer="16"/>
-<wire x1="32.385" y1="120.9675" x2="32.385" y2="43.18" width="0.254" layer="16"/>
-<wire x1="29.845" y1="123.5075" x2="32.385" y2="120.9675" width="0.254" layer="16"/>
-<wire x1="29.845" y1="133.6675" x2="29.845" y2="123.5075" width="0.254" layer="16"/>
-<wire x1="23.495" y1="133.6675" x2="29.845" y2="133.6675" width="0.254" layer="16"/>
-<wire x1="22.86" y1="134.3025" x2="23.495" y2="133.6675" width="0.254" layer="16"/>
-<wire x1="22.86" y1="136.525" x2="22.86" y2="134.3025" width="0.254" layer="16"/>
-<wire x1="21.9075" y1="136.525" x2="22.86" y2="136.525" width="0.254" layer="16"/>
-<wire x1="32.385" y1="43.18" x2="32.6" y2="43.18" width="0.254" layer="16"/>
-<wire x1="21.9075" y1="136.525" x2="21.83" y2="136.7" width="0.254" layer="16"/>
 </signal>
 <signal name="PGM_SWITCH_EN">
@@
 <contactref element="J3" pad="P$3"/>
 <contactref element="J1" pad="2"/>
-<contactref element="R1" pad="2"/>
-<wire x1="30.1625" y1="43.815" x2="30.7975" y2="43.18" width="0.254" layer="16"/>
-<wire x1="23.495" y1="43.815" x2="30.1625" y2="43.815" width="0.254" layer="16"/>
-<wire x1="30.7975" y1="43.18" x2="30.9" y2="43.18" width="0.254" layer="16"/>
-<wire x1="23.495" y1="43.815" x2="23.368" y2="43.942" width="0.254" layer="16"/>
 <wire x1="2.2225" y1="115.57" x2="2.2225" y2="123.19" width="0.254" layer="1"/>
 <wire x1="1.5875" y1="114.935" x2="2.2225" y2="115.57" width="0.254" layer="1"/>
@@
 <wire x1="2.2225" y1="123.19" x2="2.413" y2="123.19" width="0.254" layer="1"/>
 <wire x1="23.1775" y1="44.1325" x2="23.368" y2="43.942" width="0.254" layer="1"/>
+<contactref element="R6" pad="2"/>
+<wire x1="30.9" y1="43.18" x2="24.13" y2="43.18" width="0.254" layer="16"/>
+<wire x1="24.13" y1="43.18" x2="23.368" y2="43.942" width="0.254" layer="16"/>
 </signal>
 <signal name="SDA">
@@
 <via x="24.765" y="125.73" extent="1-16" drill="0.381"/>
 </signal>
+<signal name="PT_CTRL">
+<contactref element="R5" pad="1"/>
+<contactref element="U1" pad="44"/>
+<wire x1="33.83" y1="136.7" x2="33.861" y2="136.7" width="0.2032" layer="16"/>
+<wire x1="33.861" y1="136.7" x2="34.798" y2="135.763" width="0.2032" layer="16"/>
+<via x="34.798" y="135.763" extent="1-16" drill="0.508"/>
+<wire x1="34.798" y1="135.763" x2="34.798" y2="123.952" width="0.2032" layer="1"/>
+<wire x1="34.798" y1="123.952" x2="35.306" y2="123.444" width="0.2032" layer="1"/>
+<wire x1="35.306" y1="123.444" x2="35.306" y2="94.615" width="0.2032" layer="1"/>
+<wire x1="35.306" y1="94.615" x2="35.179" y2="94.488" width="0.2032" layer="1"/>
+<via x="35.179" y="94.488" extent="1-16" drill="0.508"/>
+<wire x1="35.179" y1="94.488" x2="35.179" y2="63.627" width="0.2032" layer="16"/>
+<wire x1="35.179" y1="63.627" x2="34.163" y2="62.611" width="0.2032" layer="16"/>
+<via x="34.163" y="62.611" extent="1-16" drill="0.508"/>
+<wire x1="34.163" y1="62.611" x2="34.163" y2="50.292" width="0.2032" layer="1"/>
+<wire x1="34.163" y1="50.292" x2="38.354" y2="46.101" width="0.2032" layer="1"/>
+<via x="38.354" y="46.101" extent="1-16" drill="0.508"/>
+<wire x1="38.354" y1="46.101" x2="38.354" y2="43.854" width="0.2032" layer="16"/>
+<wire x1="38.354" y1="43.854" x2="37.68" y2="43.18" width="0.2032" layer="16"/>
+</signal>
+<signal name="PT_READ_3.3V">
+<contactref element="R5" pad="2"/>
+<contactref element="R6" pad="1"/>
+<contactref element="R7" pad="2"/>
+<contactref element="U1" pad="40"/>
+<wire x1="32.6" y1="43.18" x2="32.6" y2="39.37" width="0.254" layer="16"/>
+<wire x1="32.6" y1="43.18" x2="35.98" y2="43.18" width="0.254" layer="16"/>
+<wire x1="32.6" y1="43.18" x2="32.6" y2="58" width="0.254" layer="16"/>
+<wire x1="32.6" y1="58" x2="39.37" y2="64.77" width="0.254" layer="16"/>
+<wire x1="39.37" y1="64.77" x2="39.37" y2="119.38" width="0.254" layer="16"/>
+<via x="39.37" y="119.38" extent="1-16" drill="0.508"/>
+<wire x1="39.37" y1="119.38" x2="39.37" y2="130.81" width="0.254" layer="1"/>
+<via x="39.37" y="130.81" extent="1-16" drill="0.508"/>
+<wire x1="39.37" y1="130.81" x2="29.21" y2="130.81" width="0.254" layer="16"/>
+<wire x1="29.21" y1="130.81" x2="26.797" y2="133.223" width="0.254" layer="16"/>
+<wire x1="26.797" y1="133.223" x2="26.797" y2="135.733" width="0.2032" layer="16"/>
+<wire x1="26.797" y1="135.733" x2="25.83" y2="136.7" width="0.2032" layer="16"/>
+</signal>
 </signals>

Commit message: updating switch circuit and re-routing
the pi_grammer has the isolation switch, so I am now using the onboard switch to isolate the FJ's SPI lines. This will hopefully elliminate the need for the occasional hard reset on the testbed.

Re-routing everything manually. The original design was autorouted and was pretty ugly.

Currently most of the important stuff is routed nicely. Still needs LEDs and some switch stuff routed.
Parts:
- removed JP1: MISO, SparkFun-Jumpers:SMT-JUMPER_2_NC_PASTE_NO-SILK
- removed JP2: SCK, SparkFun-Jumpers:SMT-JUMPER_2_NC_PASTE_NO-SILK
- removed JP3: RST, SparkFun-Jumpers:SMT-JUMPER_2_NC_PASTE_NO-SILK
- removed JP4: MOSI, SparkFun-Jumpers:SMT-JUMPER_2_NC_PASTE_NO-SILK
- added C1: (no value), Testing:0603-CAP
- added U$1: (no value), SparkFun:STAND-OFF-TIGHT
- U1: device Testing:FLYING_JALAPENO_V2_M -> Testing:FLYING_JALAPENO_V3_1_M
- moved U2 68.7 mm to (44.5, 58.4), turned to 0 degrees
Connections:
- net PGM_SWITCH_EN renamed SPI_SWITCH_EN
- removed net MISO_P: J1.1, JP1.1, U2.1
- removed net MOSI_P: J1.4, JP4.1, U2.11
- removed net RST_P: J1.5, JP3.1, U2.8
- removed net SCK_P: J1.3, JP2.1, U2.4
- new net CS_FJ: U1.60, U2.9
- new net MISO_FJ: U1.29, U2.2
- new net MOSI_FJ: U1.59, U2.10
- new net SCK_FJ: U1.30, U2.3
- net 5V_VIN: now also C1.1
- net CS: now also U2.8; no longer U1.60
- net GND: now also C1.2
- net MISO: now also J1.1, U2.1; no longer JP1.2, U1.29, U2.2
- net MOSI: now also J1.4, U2.11; no longer JP4.2, U1.59, U2.10
- net RST: now also J1.5; no longer JP3.2, U2.9
- net RX1_FJ: no longer J3.P$5
- net SCK: now also J1.3, U2.4; no longer JP2.2, U1.30, U2.3
- net TX1_FJ: no longer J3.P$19, J3.P$4
Routing:
- net N$6: track 186.6 -> 0.00 mm, vias 1 -> 0
- net N$5: track 180.7 -> 0.00 mm, vias 1 -> 0
- net N$4: track 171.2 -> 0.00 mm
- net N$3: track 127.4 -> 0.00 mm, vias 1 -> 0
- net PT_READ_3.3V: track 115.1 -> 7.19 mm, vias 2 -> 0
- net DTR_FJ: track 107.0 -> 0.00 mm, vias 1 -> 0
- net SCK_FJ: track 0.00 -> 104.9 mm
- net MISO_FJ: track 0.00 -> 98.5 mm
- net CS: track 115.1 -> 18.2 mm
- net PT_CTRL: track 96.6 -> 0.00 mm, vias 4 -> 0
- net CS_FJ: track 0.00 -> 92.3 mm, vias 0 -> 2
- net MOSI_FJ: track 0.00 -> 84.8 mm
- net SPI_SWITCH_EN: track 61.4 -> 98.4 mm, vias 2 -> 3
- net MOSI: track 149.6 -> 113.0 mm, vias 2 -> 0
- net SCK: track 141.6 -> 106.5 mm, vias 3 -> 1
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Other:
- board text added: "0.1uF"
- board text added: "Serial LCD 16x2 v2"
- board text added: "v2 (2/18/2019) Plewis"
- board text removed: "Serial LCD 16x2"
- board text removed: "v01 (11/15/2016) Plewis"

Commit message: finished re-routing on PB
Routing:
- net N$4: track 0.00 -> 188.2 mm, vias 0 -> 2
- net 5V_VIN: track 7.84 -> 189.1 mm, vias 0 -> 3
- net N$3: track 0.00 -> 178.7 mm, vias 0 -> 2
- net N$6: track 0.00 -> 172.0 mm, vias 0 -> 4
- net N$5: track 0.00 -> 169.0 mm, vias 0 -> 5
- net DTR_FJ: track 0.00 -> 114.5 mm, vias 0 -> 2
- net PT_CTRL: track 0.00 -> 111.1 mm, vias 0 -> 2
- net PT_READ_3.3V: track 7.19 -> 105.8 mm, vias 0 -> 4
- net MISO_FJ: track 98.5 -> 94.5 mm
- net RAW_VIA_V2: track 86.2 -> 88.2 mm
- net CS_FJ: track 92.3 -> 91.1 mm
