File: 16x2/TB EAGLE/PB/SerLCD_16x2_pb.brd (EAGLE design)
At the start: 73.7 x 139.7 mm, 20 parts, among them J1 AVR_PROG, J3 SER_LCD16X2, U1 5V Flying Jalapeno, U2 74LVC4066_MUX_1:1_X4

Commit message: 16x2 testbed PB updated for new qwiic connector version
Connections:
- net GND: no longer J3.P$18
- net RAW_VIA_V2: no longer J3.P$17
Routing:
- net RAW_VIA_V2: track 88.2 -> 81.1 mm
- net RST: track 44.2 -> 42.9 mm
Other:
- board text added: "Serial LCD 16x2 v3"
- board text added: "v3 (4/27/2020) Plewis"
- board text removed: "Serial LCD 16x2 v2"
- board text removed: "v2 (2/18/2019) Plewis"
Changed lines of the file:
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@@
 <?xml version="1.0" encoding="utf-8"?>
 <!DOCTYPE eagle SYSTEM "eagle.dtd">
-<eagle version="9.2.2">
+<eagle version="9.5.2">
 <drawing>
 <settings>
@@
 <wire x1="71.12" y1="118.11" x2="1.27" y2="118.11" width="0.254" layer="49"/>
 <wire x1="1.27" y1="118.11" x2="0" y2="115.57" width="0.254" layer="49" curve="90"/>
-<text x="34.29" y="125.73" size="1.778" layer="21" font="vector" ratio="15">Serial LCD 16x2 v2</text>
-<text x="71.882" y="61.976" size="1.27" layer="16" font="vector" ratio="15" rot="MR270">v2 (2/18/2019) Plewis</text>
+<text x="34.29" y="125.73" size="1.778" layer="21" font="vector" ratio="15">Serial LCD 16x2 v3</text>
+<text x="71.882" y="61.976" size="1.778" layer="16" font="vector" ratio="15" rot="MR270">v3 (4/27/2020) Plewis</text>
 <text x="7.366" y="4.191" size="2.286" layer="21" font="vector" ratio="15">PRETEST
    &amp;
@@
 <contactref element="J3" pad="P$1"/>
 <contactref element="J3" pad="P$2"/>
-<contactref element="J3" pad="P$18"/>
 <contactref element="J1" pad="6"/>
 <contactref element="J2" pad="6"/>
@@
 <contactref element="U1" pad="33"/>
 <contactref element="U1" pad="3"/>
-<contactref element="J3" pad="P$17"/>
 <contactref element="J3" pad="P$15"/>
 <wire x1="11.83" y1="135.208" x2="11.83" y2="130.41" width="0.508" layer="16"/>
@@
 <wire x1="30.48" y1="84.5312" x2="30.48" y2="78.74" width="0.508" layer="16"/>
 <wire x1="30.48" y1="78.74" x2="26.162" y2="74.422" width="0.508" layer="16"/>
-<wire x1="23.368" y1="84.5058" x2="30.4546" y2="84.5058" width="0.508" layer="16"/>
 <wire x1="30.4546" y1="84.5058" x2="30.48" y2="84.5312" width="0.508" layer="16"/>
 <wire x1="11.83" y1="137.208" x2="11.83" y2="135.208" width="0.508" layer="16"/>
@@
 <contactref element="J1" pad="5"/>
 <wire x1="4.953" y1="128.27" x2="8.89" y2="128.27" width="0.3048" layer="16"/>
-<wire x1="23.368" y1="113.792" x2="23.368" y2="93.98" width="0.3048" layer="16"/>
+<wire x1="23.368" y1="113.792" x2="23.368" y2="95.3516" width="0.3048" layer="16"/>
 <wire x1="8.89" y1="128.27" x2="23.368" y2="113.792" width="0.3048" layer="16"/>
 </signal>
